File: Hardware/InkTime_Schematic.brd (EAGLE design)
At the start: 46 x 35 mm, 105 parts, among them IC1 BQ25180YBGR, IC2 DRV2605YZFR, IC3 BMA421, IC9 RT6160AWSC, J1 503480-2400, J2 TC2030-IDC, J4 KH-TYPE-C-16P, Q3 SI1308EDL-T1-GE3, U1 NRF52840_QF, U3 MAX17048G+T10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

Commit message: final
Parts:
- C1, C1-EP-DR, C10, C11, C12, C13, C16, C17, C18, C19, C2, C22, C3, C4, C5, C7, C8, C9, EPD_C5: device InkTime_v5:NORDIC_NRF_3_RESC0201_L -> InkTime_v5:GRM011R60J152KE01L_2_CAPC0201X13N
- C2-EP-DR, C24, C25, C33, C39: device InkTime_v5:PERFECT_0402_0402 -> InkTime_v5:NORDIC_NRF_3_RESC0402_L
Routing:
- net GND: track 359.4 -> 364.6 mm, vias 18 -> 19
- net VBUS/1.5D: track 11.3 -> 12.1 mm
- net 3V3/2.4A: track 119.7 -> 120.4 mm
- added copper zone on layer 1, net GND
- added copper zone on layer 16, net GND
Other:
- outline, holes or cut-outs redrawn
