File: Hardware/InkTime_Schematic.sch (EAGLE design)
At the start: 105 parts, among them IC1 BQ25180YBGR, IC2 DRV2605YZFR, IC3 BMA421, IC9 RT6160AWSC, J1 503480-2400, J2 TC2030-IDC, J4 KH-TYPE-C-16P, Q3 SI1308EDL-T1-GE3, U1 NRF52840_QF, U3 MAX17048G+T10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

Commit message: final
Other:
- moved on the sheet: EPD_C10, EPD_C11, EPD_C12, EPD_C6, EPD_C8, EPD_C9
